File: keyboards/keyboards.kicad_pcb (KiCad board)
At the start: 2 copper layers, 119.6 x 98.3 mm, 34 parts, among them J1 Conn_02x08_Odd_Even, J2 Conn_02x08_Odd_Even, J3 Conn_02x08_Odd_Even, J4 Conn_02x08_Odd_Even, J5 Screw_Terminal_01x02, J6 Screw_Terminal_01x02, J7 Screw_Terminal_01x10, U1 4051, U2 4051, U3 4051, U4 4051, U5 6N138

Commit message: Files updated to Kicad 8.0
Parts:
- removed A1: Arduino_Nano_v3.x, Arduino:Arduino_Nano_Every
- removed C5: 4u7, Capacitor_SMD:C_1206_3216Metric_Pad1.42x1.75mm_HandSolder
- removed D1: D_Schottky_ALT, Resistors_SMD:R_2010_HandSoldering
- removed J5, J6: Screw_Terminal_01x02, TerminalBlock_Phoenix:TerminalBlock_Phoenix_MPT-0,5-2-2.54_1x02_P2.54mm_Horizontal
- removed J7: Screw_Terminal_01x10, TerminalBlock_Phoenix:TerminalBlock_Phoenix_MPT-0,5-10-2.54_1x10_P2.54mm_Horizontal
- removed R10: 10K, Resistor_SMD:R_2010_5025Metric_Pad1.52x2.65mm_HandSolder
- removed R11: 220, Resistor_SMD:R_2010_5025Metric_Pad1.52x2.65mm_HandSolder
- removed R9: 470, Resistor_SMD:R_2010_5025Metric_Pad1.52x2.65mm_HandSolder
- removed U5: 6N138, Package_DIP:DIP-8_W7.62mm
- added A2: Arduino_Nano_v3.x, Module:Arduino_Nano, F.Cu at (139.3, 72.6)
- C1, C2, C3, C4: footprint Capacitor_SMD:C_0805_2012Metric_Pad1.15x1.40mm_HandSolder -> Capacitor_SMD:C_1206_3216Metric_Pad1.33x1.80mm_HandSolder
- J1, J2, J3, J4: footprint Connector_Multicomp:Multicomp_MC9A12-1634_2x08_P2.54mm_Vertical -> Connector_IDC:IDC-Header_2x08_P2.54mm_Vertical
- R1, R2, R3, R4, R5, R6, R7, R8: footprint Resistor_SMD:R_2010_5025Metric_Pad1.52x2.65mm_HandSolder -> Resistor_SMD:R_1206_3216Metric_Pad1.30x1.75mm_HandSolder
- REF3: footprint Mounting_Holes:MountingHole_3mm -> MountingHole:MountingHole_3mm
- moved R2 6.93 mm to (178.0, 132.6)
- moved R7 6.55 mm to (171.5, 132.6)
- moved U2 6.30 mm to (178.3, 122.2)
- moved U4 6.30 mm to (123.9, 122.2)
- moved C2 6.30 mm to (166.2, 123.2)
- moved C4 6.30 mm to (111.6, 123.2)
- moved R8 5.90 mm to (116.9, 132.6)
- moved R4 5.82 mm to (123.0, 132.6)
- moved R1 5.74 mm to (178.5, 81.8)
- moved R5 5.56 mm to (171.5, 81.8)
- moved R3 4.20 mm to (123.3, 81.8)
- moved R6 4.20 mm to (116.9, 81.8)
- moved C1 3.44 mm to (166.3, 73.5)
- moved C3 3.44 mm to (111.8, 73.5)
- moved U1 3.44 mm to (178.3, 72.4)
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Routing:
- net /SCK: track 130.4 -> 0.00 mm
- net /SS4: track 109.6 -> 0.00 mm
- net /MISO: track 96.7 -> 0.00 mm
- net /MOSI: track 93.6 -> 0.00 mm, vias 1 -> 0
- net /SS3: track 85.5 -> 0.00 mm
- net /SS2: track 84.0 -> 0.00 mm
- net /SS1: track 81.8 -> 0.00 mm
- net /MKB3: track 127.8 -> 46.8 mm, vias 0 -> 1
- net +9V: track 77.7 -> 0.00 mm
- net /T7: track 253.7 -> 204.5 mm, vias 1 -> 0
- net +5V: track 235.5 -> 186.5 mm
- net Net-(D1-Pad2): track 48.9 -> 0.00 mm
- net /MKB: track 95.3 -> 53.1 mm
- net GND: track 373.6 -> 333.5 mm
- net Net-(A1-Pad2): track 39.8 -> 0.00 mm
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Other:
- net class Default removed
- net class Power removed
- board text added: "Keyboards Control"
- board text added: "Left section"
- board text added: "Right section"
- board text added: "V1.1"
- board text removed: "+5V"
- board text removed: "+9V"
- board text removed: "2"
- board text removed: "GND"
- board text removed: "Keyboards and Pedals"
- board text removed: "MISO"
- board text removed: "MOSI"
- board text removed: "Pedals MIDI"
- board text removed: "SCK"
- board text removed: "SPI"
- board text removed: "SS1"
- board text removed: "SS2"
- board text removed: "SS3"
- board text removed: "SS4"
- board text removed: "V1.0"
