File: keyboards/keyboards.kicad_sch (KiCad schematic)
At the start: 30 parts, among them J1 Conn_02x08_Odd_Even, J2 Conn_02x08_Odd_Even, J3 Conn_02x08_Odd_Even, J4 Conn_02x08_Odd_Even, J5 Screw_Terminal_01x02, J6 Screw_Terminal_01x02, J7 Screw_Terminal_01x10, U1 4051, U2 4051, U3 4051, U4 4051, U5 6N138

Commit message: Files updated to Kicad 8.0
Parts:
- removed A1: Arduino_Nano_v3.x, Arduino:Arduino_Nano_Every, symbol keyboards-rescue:Arduino_Nano_v3.x-MCU_Module-keyboards_pedals-rescue
- removed C5: 4u7, Capacitor_SMD:C_1206_3216Metric_Pad1.42x1.75mm_HandSolder, symbol Device:C
- removed D1: D_Schottky_ALT, Resistors_SMD:R_2010_HandSoldering, symbol Device:D_Schottky_ALT
- removed J5, J6: Screw_Terminal_01x02, TerminalBlock_Phoenix:TerminalBlock_Phoenix_MPT-0,5-2-2.54_1x02_P2.54mm_Horizontal, symbol Connector:Screw_Terminal_01x02
- removed J7: Screw_Terminal_01x10, TerminalBlock_Phoenix:TerminalBlock_Phoenix_MPT-0,5-10-2.54_1x10_P2.54mm_Horizontal, symbol Connector:Screw_Terminal_01x10
- removed R10: 10K, Resistor_SMD:R_2010_5025Metric_Pad1.52x2.65mm_HandSolder, symbol Device:R
- removed R11: 220, Resistor_SMD:R_2010_5025Metric_Pad1.52x2.65mm_HandSolder, symbol Device:R
- removed R9: 470, Resistor_SMD:R_2010_5025Metric_Pad1.52x2.65mm_HandSolder, symbol Device:R
- removed U5: 6N138, Package_DIP:DIP-8_W7.62mm, symbol Isolator:6N138
- added A2: Arduino_Nano_v3.x, Module:Arduino_Nano, symbol MCU_Module:Arduino_Nano_v3.x
- C1, C2, C3, C4: footprint Capacitor_SMD:C_0805_2012Metric_Pad1.15x1.40mm_HandSolder -> Capacitor_SMD:C_1206_3216Metric_Pad1.33x1.80mm_HandSolder
- J1, J2, J3, J4: footprint Connector_Multicomp:Multicomp_MC9A12-1634_2x08_P2.54mm_Vertical -> Connector_IDC:IDC-Header_2x08_P2.54mm_Vertical
- R1, R2, R3, R4, R5, R6, R7, R8: footprint Resistor_SMD:R_2010_5025Metric_Pad1.52x2.65mm_HandSolder -> Resistor_SMD:R_1206_3216Metric_Pad1.30x1.75mm_HandSolder
Connections:
- net +5V: now also A2.27 (+5V)
- net BRA: now also A2.1 (D1/TX)
- net BRB: now also A2.5 (D2)
- net GND: now also A2.29 (GND), A2.4 (GND)
- net MKA: now also A2.6 (D3)
- net MKB: now also A2.7 (D4)
- net MUX_A1: now also A2.8 (D5)
- net MUX_A2: now also A2.9 (D6)
- net MUX_A3: now also A2.10 (D7)
- net T0: now also A2.19 (A0)
- net T1: now also A2.20 (A1)
- net T2: now also A2.21 (A2)
- net T3: now also A2.22 (A3)
- net T4: now also A2.23 (A4)
- net T5: now also A2.24 (A5)
- net T6: now also A2.25 (A6)
- net T7: now also A2.26 (A7)
- no-connect marks 3 -> 12
Other:
- note added: "Left section"
- note added: "Right section"
- note removed: "EXT. PS"
- note removed: "Pedal MIDI"
- note removed: "SPI"
- company: Clone Hammond B3 / setBfree MIDI controls -> Picherie
- title: Keyboards and pedals control -> Keyboards control
- moved on the sheet: C1, C2, C3, C4, J1, J2, J3, J4, R1, R2, R3, R4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
