File: volume_reverb_overdrive/volume_reverb_overdrive.kicad_sch (KiCad schematic)
At the start: 17 parts, among them J1 Conn_02x05_Odd_Even, SW1 RotaryEncoder, SW2 RotaryEncoder, SW3 RotaryEncoder_Switch, U1 74HC14

Commit message: New organ architecture with mother board
Changed lines of the file:
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@@
 (kicad_sch
-	(version 20231120)
+	(version 20250114)
 	(generator "eeschema")
-	(generator_version "8.0")
+	(generator_version "9.0")
 	(paper "A4")
 	(title_block
@@
 		(company "Picherie")
 	)
+	(text "GPIO 17"
+		(exclude_from_sim no)
+		(at 195.58 139.7 0)
+		(effects
+			(font
+				(size 1.27 1.27)
+			)
+			(justify left bottom)
+		)
+	)
+	(text "RPI SHUT DOWN DEBOUNCE"
+		(exclude_from_sim no)
+		(at 88.9 106.68 0)
+		(effects
+			(font
+				(size 3 3)
+			)
+			(justify right bottom)
+		)
+	)
+	(text "REVERB"
+		(exclude_from_sim no)
+		(at 86.106 36.576 0)
+		(effects
+			(font
+				(size 3 3)
+			)
+			(justify left bottom)
+		)
+	)
+	(text "GPIO 25"
+		(exclude_from_sim no)
+		(at 138.43 142.24 0)
+		(effects
+			(font
+				(size 1.27 1.27)
+			)
+			(justify left bottom)
+		)
+	)
+	(text "to GPIO 24 (RPI pin 18 / Pi-DAC+ volume control)"
+		(exclude_from_sim no)
+		(at 95.25 139.7 0)
+		(effects
+			(font
+				(size 1.27 1.27)
+			)
+			(justify left bottom)
+		)
+	)
+	(text "OVERDRIVE / RPI SHUTDOWN"
+		(exclude_from_sim no)
+		(at 121.92 29.21 0)
+		(effects
+			(font
+				(size 3 3)
+			)
+			(justify left bottom)
+		)
+	)
+	(text "to GPIO 23 (RPI pin 16 / Pi-DAC+ volume control)"
+		(exclude_from_sim no)
+		(at 95.25 137.16 0)
+		(effects
+			(font
+				(size 1.27 1.27)
+			)
+			(justify left bottom)
+		)
+	)
+	(text "VOLUME"
+		(exclude_from_sim no)
+		(at 48.006 36.576 0)
+		(effects
+			(font
+				(size 3 3)
+			)
+			(justify right bottom)
+		)
+	)
+	(text "GPIO 26"
+		(exclude_from_sim no)
+		(at 195.58 142.24 0)
+		(effects
+			(font
+				(size 1.27 1.27)
+			)
+			(justify left bottom)
+		)
+	)
+	(text "GPIO 16"
+		(exclude_from_sim no)
+		(at 195.58 137.16 0)
+		(effects
+			(font
+				(size 1.27 1.27)
+			)
+			(justify left bottom)
+		)
+	)
 	(junction
 		(at 154.94 57.15)
@@
 		)
 	)
-	(text "GPIO 17"
-		(exclude_from_sim no)
-		(at 195.58 139.7 0)
-		(effects
-			(font
-				(size 1.27 1.27)
-			)
-			(justify left bottom)
-		)
-	)
-	(text "RPI SHUT DOWN DEBOUNCE"
-		(exclude_from_sim no)
-		(at 88.9 106.68 0)
-		(effects
-			(font
-				(size 3 3)
-			)
-			(justify right bottom)
-		)
-	)
-	(text "REVERB"
-		(exclude_from_sim no)
-		(at 86.106 36.576 0)
-		(effects
-			(font
-				(size 3 3)
-			)
-			(justify left bottom)
-		)
-	)
-	(text "GPIO 25"
-		(exclude_from_sim no)
-		(at 138.43 142.24 0)
-		(effects
-			(font
-				(size 1.27 1.27)
-			)
-			(justify left bottom)
-		)
-	)
-	(text "to GPIO 24 (RPI pin 18 / Pi-DAC+ volume control)"
-		(exclude_from_sim no)
-		(at 95.25 139.7 0)
-		(effects
-			(font
-				(size 1.27 1.27)
-			)
-			(justify left bottom)
-		)
-	)
-	(text "OVERDRIVE / RPI SHUTDOWN"
-		(exclude_from_sim no)
-		(at 121.92 29.21 0)
-		(effects
-			(font
-				(size 3 3)
-			)
-			(justify left bottom)
-		)
-	)
-	(text "to GPIO 23 (RPI pin 16 / Pi-DAC+ volume control)"
-		(exclude_from_sim no)
-		(at 95.25 137.16 0)
-		(effects
-			(font
-				(size 1.27 1.27)
-			)
-			(justify left bottom)
-		)
-	)
-	(text "VOLUME"
-		(exclude_from_sim no)
-		(at 48.006 36.576 0)
-		(effects
-			(font
-				(size 3 3)
-			)
-			(justify right bottom)
-		)
-	)
-	(text "GPIO 26"
-		(exclude_from_sim no)
-		(at 195.58 142.24 0)
-		(effects
-			(font
-				(size 1.27 1.27)
-			)
-			(justify left bottom)
-		)
-	)
-	(text "GPIO 16"
-		(exclude_from_sim no)
-		(at 195.58 137.16 0)
-		(effects
-			(font
-				(size 1.27 1.27)
-			)
-			(justify left bottom)
-		)
-	)
 	(label "OVERDRIVE_A"
 		(at 181.61 137.16 0)
-		(fields_autoplaced yes)
 		(effects
 			(font
@@
 	(label "VOLUME_B"
 		(at 157.48 139.7 180)
-		(fields_autoplaced yes)
 		(effects
 			(font
@@
 	(label "REVERB_B"
 		(at 99.06 57.15 0)
-		(fields_autoplaced yes)
 		(effects
 			(font
@@
 	(label "OVERDRIVE_B"
 		(at 158.75 57.15 0)
-		(fields_autoplaced yes)
 		(effects
 			(font
@@
 	(label "RPI_OFF"
 		(at 49.53 146.05 180)
-		(fields_autoplaced yes)
 		(effects
 			(font
@@
 	(label "OVERDRIVE_A"
 		(at 146.05 57.15 180)
-		(fields_autoplaced yes)
 		(effects
 			(font
@@
 	(label "VOLUME_A"
 		(at 33.02 55.88 180)
-		(fields_autoplaced yes)
 		(effects
 			(font
@@
 	(label "REVERB_B"
 		(at 181.61 142.24 0)
-		(fields_autoplaced yes)
 		(effects
 			(font
@@
 	(label "OVERDRIVE_B"
 		(at 181.61 139.7 0)
-		(fields_autoplaced yes)
 		(effects
 			(font
@@
 	(label "VOLUME_A"
 		(at 157.48 137.16 180)
-		(fields_autoplaced yes)
 		(effects
 			(font
@@
 	(label "REVERB_A"
 		(at 157.48 142.24 180)
-		(fields_autoplaced yes)
 		(effects
 			(font
@@
 	(label "RPI_OFF"
 		(at 146.05 35.56 180)
-		(fields_autoplaced yes)
 		(effects
 			(font
@@
 	(label "VOLUME_B"
 		(at 45.72 55.88 0)
-		(fields_autoplaced yes)
 		(effects
 			(font
@@
 	(label "SHUT_DOWN"
 		(at 88.9 134.62 0)
-		(fields_autoplaced yes)
 		(effects
 			(font
@@
 	(label "REVERB_A"
 		(at 87.63 57.15 180)
-		(fields_autoplaced yes)
 		(effects
 			(font
@@
 		(at 81.28 134.62 0)
 		(unit 1)
-		(exclude_from_sim yes)
+		(exclude_from_sim no)
 		(in_bom yes)
 		(on_board yes)
@@
 		)
 	)
+	(embedded_fonts no)
 )
